File: h-bridge-setup.kicad_sch (KiCad schematic)
At the start: 8 parts, among them U11 SN754410NE

Commit message: scematics and basic PCB layout
Parts:
- removed C12: 100 µF, Capacitor_THT:CP_Radial_D6.3mm_P2.50mm, symbol Device:C_Polarized
Other:
- moved on the sheet: R11
Changed lines of the file:
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@@
 	(paper "A4")
-	(junction
-		(at 118.11 54.61)
-		(diameter 0)
-		(color 0 0 0 0)
-	)
 	(junction
 		(at 118.11 67.31)
@@
 	)
 	(junction
-		(at 125.73 67.31)
-		(diameter 0)
-		(color 0 0 0 0)
-	)
-	(junction
 		(at 97.79 73.66)
 		(diameter 0)
@@
 	(wire
 		(pts
-			(xy 81.28 76.2) (xy 81.28 86.36)
+			(xy 71.12 85.09) (xy 71.12 86.36)
 		)
 		(stroke
@@
 	(wire
 		(pts
-			(xy 69.85 72.39) (xy 86.36 72.39)
-		)
-		(stroke
-			(width 0)
-			(type default)
-		)
-	)
-	(wire
-		(pts
-			(xy 69.85 76.2) (xy 81.28 76.2)
-		)
-		(stroke
-			(width 0)
-			(type default)
-		)
-	)
-	(wire
-		(pts
-			(xy 125.73 54.61) (xy 125.73 67.31)
+			(xy 69.85 78.74) (xy 88.9 78.74)
+		)
+		(stroke
+			(width 0)
+			(type default)
+		)
+	)
+	(wire
+		(pts
+			(xy 69.85 85.09) (xy 71.12 85.09)
 		)
 		(stroke
@@
 	(wire
 		(pts
-			(xy 69.85 68.58) (xy 78.74 68.58)
+			(xy 69.85 74.93) (xy 78.74 74.93)
 		)
 		(stroke
@@
 	(wire
 		(pts
-			(xy 88.9 68.58) (xy 86.36 68.58)
+			(xy 88.9 74.93) (xy 86.36 74.93)
 		)
 		(stroke
@@
 	(wire
 		(pts
-			(xy 78.74 80.01) (xy 78.74 88.9)
-		)
-		(stroke
-			(width 0)
-			(type default)
-		)
-	)
-	(wire
-		(pts
 			(xy 157.48 77.47) (xy 157.48 76.2)
 		)
@@
 	(wire
 		(pts
-			(xy 88.9 68.58) (xy 88.9 76.2)
+			(xy 88.9 74.93) (xy 88.9 76.2)
 		)
 		(stroke
@@
 	(wire
 		(pts
-			(xy 78.74 88.9) (xy 91.44 88.9)
+			(xy 71.12 86.36) (xy 82.55 86.36)
 		)
 		(stroke
@@
 	(wire
 		(pts
-			(xy 69.85 80.01) (xy 78.74 80.01)
+			(xy 69.85 88.9) (xy 91.44 88.9)
 		)
 		(stroke
@@
 	(wire
 		(pts
-			(xy 86.36 78.74) (xy 86.36 72.39)
-		)
-		(stroke
-			(width 0)
-			(type default)
-		)
-	)
-	(wire
-		(pts
-			(xy 118.11 46.99) (xy 118.11 54.61)
-		)
-		(stroke
-			(width 0)
-			(type default)
-		)
-	)
-	(wire
-		(pts
 			(xy 130.81 86.36) (xy 158.75 86.36)
 		)
@@
 	(wire
 		(pts
-			(xy 81.28 86.36) (xy 82.55 86.36)
-		)
-		(stroke
-			(width 0)
-			(type default)
-		)
-	)
-	(wire
-		(pts
 			(xy 130.81 73.66) (xy 158.75 73.66)
 		)
@@
 	(wire
 		(pts
-			(xy 88.9 78.74) (xy 86.36 78.74)
-		)
-		(stroke
-			(width 0)
-			(type default)
-		)
-	)
-	(wire
-		(pts
 			(xy 100.33 78.74) (xy 96.52 78.74)
 		)
@@
 	(wire
 		(pts
-			(xy 118.11 54.61) (xy 118.11 67.31)
+			(xy 118.11 46.99) (xy 118.11 67.31)
 		)
 		(stroke
@@
 	(hierarchical_label "1A"
 		(shape input)
-		(at 69.85 68.58 180)
+		(at 69.85 74.93 180)
 		(fields_autoplaced yes)
 		(effects
@@
 		)
 		(property "Netclass" "LOGIC_3V3"
-			(at 69.85 69.85 0)
+			(at 69.85 76.2 0)
 			(effects
 				(font
@@
 	(hierarchical_label "2A"
 		(shape input)
-		(at 69.85 72.39 180)
+		(at 69.85 78.74 180)
 		(fields_autoplaced yes)
 		(effects
@@
 		)
 		(property "Netclass" "LOGIC_3V3"
-			(at 69.85 73.66 0)
+			(at 69.85 80.01 0)
 			(effects
 				(font
@@
 	(hierarchical_label "3A"
 		(shape input)
-		(at 69.85 76.2 180)
+		(at 69.85 85.09 180)
 		(fields_autoplaced yes)
 		(effects
@@
 		)
 		(property "Netclass" "LOGIC_3V3"
-			(at 69.85 77.47 0)
+			(at 69.85 86.36 0)
 			(effects
 				(font
@@
 	(hierarchical_label "4A"
 		(shape input)
-		(at 69.85 80.01 180)
+		(at 69.85 88.9 180)
 		(fields_autoplaced yes)
 		(effects
@@
 		)
 		(property "Netclass" "LOGIC_3V3"
-			(at 69.85 81.28 0)
+			(at 69.85 90.17 0)
 			(effects
 				(font
@@
 	)
 	(symbol
-		(lib_id "Device:C_Polarized")
-		(at 121.92 54.61 90)
-		(unit 1)
-		(exclude_from_sim no)
-		(in_bom yes)
-		(on_board yes)
-		(dnp no)
-		(property "Reference" "C12"
-			(at 121.031 46.99 90)
-			(effects
-				(font
-					(size 1.27 1.27)
-				)
-			)
-		)
-		(property "Value" "100 µF"
-			(at 121.92 49.53 90)
-			(effects
-				(font
-					(size 1.27 1.27)
-				)
-			)
-		)
-		(property "Footprint" "Capacitor_THT:CP_Radial_D6.3mm_P2.50mm"
-			(at 125.73 53.6448 0)
-			(effects
-				(font
-					(size 1.27 1.27)
-				)
-				(hide yes)
-			)
-		)
-		(property "Datasheet" "~"
-			(at 121.92 54.61 0)
-			(effects
-				(font
-					(size 1.27 1.27)
-				)
-				(hide yes)
-			)
-		)
-		(property "Description" "Polarized capacitor"
-			(at 121.92 54.61 0)
-			(effects
-				(font
-					(size 1.27 1.27)
-				)
-				(hide yes)
-			)
-		)
-		(pin "2"
-		)
-		(pin "1"
-		)
-		(instances
-			(project "WeichenBaustein"
-				(path "/1725eceb-0961-4b11-ba66-d87e36cc49b0/870002fe-9ed7-4fd7-af42-f8cf7009dfee"
-					(reference "C12")
-					(unit 1)
-				)
-				(path "/1725eceb-0961-4b11-ba66-d87e36cc49b0/908cb60b-c7ff-4b0f-bb0a-ce4cf7cc4c78"
-					(reference "C32")
-					(unit 1)
-				)
-				(path "/1725eceb-0961-4b11-ba66-d87e36cc49b0/a4def09f-05e5-4062-9e88-4e7ecfe08a37"
-					(reference "C42")
-					(unit 1)
-				)
-				(path "/1725eceb-0961-4b11-ba66-d87e36cc49b0/b1af24be-8e4d-49d7-bd98-42c545b755d4"
-					(reference "C22")
-					(unit 1)
-				)
-			)
-		)
-	)
-	(symbol
 		(lib_id "power:GND")
 		(at 105.41 67.31 270)
@@
 	(symbol
 		(lib_id "Device:R")
-		(at 82.55 68.58 270)
+		(at 82.55 74.93 270)
 		(unit 1)
 		(exclude_from_sim no)
@@
 		(dnp no)
 		(property "Reference" "R11"
-			(at 82.55 68.58 90)
+			(at 82.55 74.93 90)
 			(effects
 				(font
@@
 		)
 		(property "Value" "100R"
-			(at 82.55 66.294 90)
+			(at 82.55 72.644 90)
 			(effects
 				(font
@@
 		)
 		(property "Footprint" "Resistor_SMD:R_1206_3216Metric_Pad1.30x1.75mm_HandSolder"
-			(at 82.55 66.802 90)
+			(at 82.55 73.152 90)
 			(effects
 				(font
@@
 		)
 		(property "Datasheet" "~"
-			(at 82.55 68.58 0)
+			(at 82.55 74.93 0)
 			(effects
 				(font
@@
 		)
 		(property "Description" "Resistor"
-			(at 82.55 68.58 0)
-			(effects
-				(font
+			(at 82.55 74.93 0)
+			(effects
+				(font

Commit message: basic routing
Parts:
- removed R11, R12, R13, R14: 100R, Resistor_SMD:R_1206_3216Metric_Pad1.30x1.75mm_HandSolder, symbol Device:R
Connections:
- net 1A: now also U11.2 (1A)
- net 2A: now also U11.7 (2A)
- net 3A: now also U11.10 (3A)
- net 4A: now also U11.15 (4A)
- net W1_B: now also U11.6 (2Y); no longer U11.3 (1Y)
- net W1_R: now also U11.3 (1Y); no longer U11.6 (2Y)
- net W2_B: now also U11.14 (4Y); no longer U11.11 (3Y)
- net W2_R: now also U11.11 (3Y); no longer U11.14 (4Y)
