File: WeichenBaustein.kicad_sch (KiCad schematic)
At the start: 8 parts, among them J1 Conn_01x16, J7 Conn_01x12_Female, U2 esp32_dev4_left, U3 esp32_dev4_right

Commit message: scematics and basic PCB layout
Parts:
- removed J1: Conn_01x16, symbol Connector_Generic:Conn_01x16
- removed J7: Conn_01x12_Female, Custom:1729225, symbol Connector:Conn_01x12_Female
- added C12: 100 µF, Capacitor_THT:CP_Radial_D6.3mm_P2.50mm, symbol Device:C_Polarized
- added J1: Conn_01x08, Custom:1729186, symbol Connector_Generic:Conn_01x08
- added J2: 1726150, 1726150, symbol Custom:1726150
- U2: footprint fp_esp32_dev4:esp32_dev_left -> Custom:esp32_dev_left
- U3: footprint fp_esp32_dev4:esp32_dev4_right -> Custom:esp32_dev4_right
Connections:
- net +12V: now also C12.1, J1.5 (Pin_5), J1.6 (Pin_6)
- net +5V: now also J1.1 (Pin_1), J1.2 (Pin_2)
- net GND: now also C12.2, J1.3 (Pin_3), J1.4 (Pin_4), J1.7 (Pin_7), J1.8 (Pin_8)
- net H-Bridge-setup1/W1_B: now also J2.1
- net H-Bridge-setup1/W1_R: now also J2.2
- net H-Bridge-setup1/W2_B: now also J2.3
- net H-Bridge-setup1/W2_R: now also J2.4
- net H-Bridge-setup2/W1_B: now also J2.5
- net H-Bridge-setup2/W1_R: now also J2.6
- net H-Bridge-setup2/W2_B: now also J2.7
- net H-Bridge-setup2/W2_R: now also J2.8
- net H-Bridge-setup3/W1_B: now also J2.9
- net H-Bridge-setup3/W1_R: now also J2.10
- net H-Bridge-setup3/W2_B: now also J2.11
- net H-Bridge-setup3/W2_R: now also J2.12
- net H-Bridge-setup4/W1_B: now also J2.13
- net H-Bridge-setup4/W1_R: now also J2.14
- net H-Bridge-setup4/W2_B: now also J2.15
- net H-Bridge-setup4/W2_R: now also J2.16

Commit message: final design
Parts:
- removed H1: MountingHole, MountingHole:MountingHole_4.3mm_M4, symbol Mechanical:MountingHole
- renumbered C12 to C1
Changed lines of the file:
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@@
 		(dnp no)
 		(fields_autoplaced yes)
-		(property "Reference" "C12"
-			(at 33.02 62.6109 0)
-			(show_name no)
-			(do_not_autoplace no)
-			(effects
-				(font
-					(size 1.27 1.27)
-				)
-				(justify right)
+		(property "Reference" "C1"
+			(at 40.64 62.6109 0)
+			(show_name no)
+			(do_not_autoplace no)
+			(effects
+				(font
+					(size 1.27 1.27)
+				)
+				(justify left)
 			)
 		)
 		(property "Value" "100 µF"
-			(at 33.02 65.1509 0)
-			(show_name no)
-			(do_not_autoplace no)
-			(effects
-				(font
-					(size 1.27 1.27)
-				)
-				(justify right)
+			(at 40.64 65.1509 0)
+			(show_name no)
+			(do_not_autoplace no)
+			(effects
+				(font
+					(size 1.27 1.27)
+				)
+				(justify left)
 			)
 		)
@@
 			(project "WeichenBaustein"
 				(path "/1725eceb-0961-4b11-ba66-d87e36cc49b0"
-					(reference "C12")
+					(reference "C1")
 					(unit 1)
 				)
@@
 					(unit 1)
 				)
-			)
-		)
-	)
-	(symbol
-		(lib_id "Mechanical:MountingHole")
-		(at 53.34 137.16 0)
-		(unit 1)
-		(body_style 1)
-		(exclude_from_sim no)
-		(in_bom yes)
-		(on_board yes)
-		(in_pos_files yes)
-		(dnp no)
-		(fields_autoplaced yes)
-		(property "Reference" "H1"
-			(at 55.88 136.525 0)
-			(show_name no)
-			(do_not_autoplace no)
-			(effects
-				(font
-					(size 1.27 1.27)
-				)
-				(justify left)
-			)
-		)
-		(property "Value" "MountingHole"
-			(at 55.88 139.065 0)
-			(show_name no)
-			(do_not_autoplace no)
-			(effects
-				(font
-					(size 1.27 1.27)
-				)
-				(justify left)
-			)
-		)
-		(property "Footprint" "MountingHole:MountingHole_4.3mm_M4"
-			(at 53.34 137.16 0)
-			(hide yes)
-			(show_name no)
-			(do_not_autoplace no)
-			(effects
-				(font
-					(size 1.27 1.27)
-				)
-			)
-		)
-		(property "Datasheet" ""
-			(at 53.34 137.16 0)
-			(hide yes)
-			(show_name no)
-			(do_not_autoplace no)
-			(effects
-				(font
-					(size 1.27 1.27)
-				)
-			)
-		)
-		(property "Description" ""
-			(at 53.34 137.16 0)
-			(show_name no)
-			(do_not_autoplace no)
-			(effects
-				(font
-					(size 1.27 1.27)
-				)
-			)
-		)
-		(instances
-			(project "WeichenBaustein"
-				(path "/1725eceb-0961-4b11-ba66-d87e36cc49b0"
-					(reference "H1")
-					(unit 1)
-				)
