File: WeichenBaustein.kicad_pcb (KiCad board)
At the start: 2 copper layers, 36 parts, among them U11 SN754410NE, U21 SN754410NE, U31 SN754410NE, U41 SN754410NE

Commit message: scematics and basic PCB layout
Parts:
- removed C22, C32, C42: 100 µF, Capacitor_THT:CP_Radial_D6.3mm_P2.50mm
- added J1: Conn_01x08, Custom:1729186, F.Cu at (161.5, 25.1)
- added J2: 1726150, Custom:1726150, F.Cu at (249.7, 32.7)
- added U2: esp32_dev4_left, Custom:esp32_dev_left, F.Cu at (180.9, 20.8)
- added U3: esp32_dev4_right, Custom:esp32_dev4_right, F.Cu at (197.4, 20.8)
- C11, C13, C21, C23, C31, C33, C41, C43, R11, R12, R13, R14, R21, R22, R23, R24, R31, R32, R33, R34, R41, R42, R43, R44: moved to B.Cu
- moved H4 187.1 mm to (250.2, 79.0)
- moved H1 184.3 mm to (250.7, 23.9)
- moved U41 133.1 mm to (221.2, 58.4)
- moved H3 127.2 mm to (176.8, 23.9)
- moved C41 125.7 mm to (226.1, 62.2), turned to -90 degrees
- moved C43 120.7 mm to (224.0, 72.4), turned to -90 degrees
- moved U11 120.7 mm to (207.5, 26.7)
- moved C11 114.6 mm to (212.3, 30.5), turned to -90 degrees
- moved C13 109.2 mm to (210.3, 40.6), turned to -90 degrees
- moved U31 106.7 mm to (221.2, 26.7)
- moved C12 105.7 mm to (200.7, 43.7)
- moved C31 102.0 mm to (226.1, 30.5), turned to -90 degrees
- moved C33 96.2 mm to (224.0, 40.6), turned to -90 degrees
- moved U21 93.7 mm to (207.5, 58.4)
- moved R44 90.4 mm to (174.8, 40.4), turned to 180 degrees
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Routing:
- net +5V: track 0.00 -> 262.0 mm, vias 0 -> 1
- net +12V: track 0.00 -> 159.1 mm
- net GND: track 0.00 -> 130.9 mm, vias 0 -> 8
- net Net-(U41-4A): track 0.00 -> 90.8 mm, vias 0 -> 1
- net Net-(U41-3A): track 0.00 -> 86.0 mm, vias 0 -> 1
- net Net-(U41-2A): track 0.00 -> 71.6 mm, vias 0 -> 1
- net Net-(U31-4A): track 0.00 -> 66.7 mm, vias 0 -> 3
- net Net-(U31-3A): track 0.00 -> 59.4 mm, vias 0 -> 1
- net Net-(U21-3A): track 0.00 -> 58.3 mm, vias 0 -> 1
- net Net-(U41-1A): track 0.00 -> 57.3 mm, vias 0 -> 3
- net /H-Bridge-setup1/W1_R: track 0.00 -> 57.3 mm, vias 0 -> 1
- net Net-(U11-3A): track 0.00 -> 57.1 mm, vias 0 -> 3
- net Net-(U11-4A): track 0.00 -> 54.7 mm, vias 0 -> 2
- net /H-Bridge-setup2/W1_R: track 0.00 -> 54.0 mm
- net /H-Bridge-setup1/W2_R: track 0.00 -> 52.1 mm, vias 0 -> 1
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- added copper zone on B.Cu, net GND
- added copper zone on F.Cu, net GND
Other:
- board outline added: 99.6 x 64.3 mm
- board text added: "${REFERENCE}"

Commit message: basic routing
Parts:
- removed R11, R12, R13, R14, R21, R22, R23, R24, R31, R32, R33, R34, R41, R42, R43, R44: 100R, Resistor_SMD:R_1206_3216Metric_Pad1.30x1.75mm_HandSolder
- moved J2 70.6 mm to (226.4, 99.3), turned to 180 degrees
- moved C12 36.9 mm to (163.8, 44.6), turned to 90 degrees
- moved H4 28.1 mm to (235.5, 102.9)
- moved H2 25.8 mm to (150.6, 102.9)
- moved H3 13.7 mm to (163.1, 23.9)
- moved H1 12.3 mm to (247.7, 11.9)
- moved C41 9.95 mm to (235.5, 58.9)
- moved C31 9.40 mm to (235.5, 30.5)
- moved J1 8.65 mm to (152.9, 25.7)
- moved C23 6.06 mm to (205.2, 69.1)
- moved C21 6.05 mm to (217.4, 58.9)
- moved U41 5.43 mm to (225.6, 55.1)
- moved C11 5.08 mm to (217.4, 30.5)
- moved C13 5.08 mm to (205.2, 40.6)
- moved U31 4.32 mm to (225.6, 26.7)
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Connections:
- U11 pad 10: Net-(U11-3A) -> /H-Bridge-setup1/3A
- U11 pad 11: /H-Bridge-setup1/W2_B -> /H-Bridge-setup1/W2_R
- U11 pad 14: /H-Bridge-setup1/W2_R -> /H-Bridge-setup1/W2_B
- U11 pad 15: Net-(U11-4A) -> /H-Bridge-setup1/4A
- U11 pad 2: Net-(U11-1A) -> /H-Bridge-setup1/1A
- U11 pad 3: /H-Bridge-setup1/W1_B -> /H-Bridge-setup1/W1_R
- U11 pad 6: /H-Bridge-setup1/W1_R -> /H-Bridge-setup1/W1_B
- U11 pad 7: Net-(U11-2A) -> /H-Bridge-setup1/2A
- U21 pad 10: Net-(U21-3A) -> /H-Bridge-setup2/3A
- U21 pad 11: /H-Bridge-setup2/W2_B -> /H-Bridge-setup2/W2_R
- U21 pad 14: /H-Bridge-setup2/W2_R -> /H-Bridge-setup2/W2_B
- U21 pad 15: Net-(U21-4A) -> /H-Bridge-setup2/4A
- U21 pad 2: Net-(U21-1A) -> /H-Bridge-setup2/1A
- U21 pad 3: /H-Bridge-setup2/W1_B -> /H-Bridge-setup2/W1_R
- U21 pad 6: /H-Bridge-setup2/W1_R -> /H-Bridge-setup2/W1_B
- U21 pad 7: Net-(U21-2A) -> /H-Bridge-setup2/2A
- U31 pad 10: Net-(U31-3A) -> /H-Bridge-setup3/3A
- U31 pad 11: /H-Bridge-setup3/W2_B -> /H-Bridge-setup3/W2_R
- U31 pad 14: /H-Bridge-setup3/W2_R -> /H-Bridge-setup3/W2_B
- U31 pad 15: Net-(U31-4A) -> /H-Bridge-setup3/4A
- U31 pad 2: Net-(U31-1A) -> /H-Bridge-setup3/1A
- U31 pad 3: /H-Bridge-setup3/W1_B -> /H-Bridge-setup3/W1_R
- U31 pad 6: /H-Bridge-setup3/W1_R -> /H-Bridge-setup3/W1_B
- U31 pad 7: Net-(U31-2A) -> /H-Bridge-setup3/2A
- U41 pad 10: Net-(U41-3A) -> /H-Bridge-setup4/3A
- U41 pad 11: /H-Bridge-setup4/W2_B -> /H-Bridge-setup4/W2_R
- U41 pad 14: /H-Bridge-setup4/W2_R -> /H-Bridge-setup4/W2_B
- U41 pad 15: Net-(U41-4A) -> /H-Bridge-setup4/4A
- U41 pad 2: Net-(U41-1A) -> /H-Bridge-setup4/1A
- U41 pad 3: /H-Bridge-setup4/W1_B -> /H-Bridge-setup4/W1_R
- U41 pad 6: /H-Bridge-setup4/W1_R -> /H-Bridge-setup4/W1_B
- U41 pad 7: Net-(U41-2A) -> /H-Bridge-setup4/2A
Routing:
- net +5V: track 262.0 -> 64.6 mm, vias 1 -> 0
- net +12V: track 159.1 -> 20.0 mm
- net GND: track 130.9 -> 10.2 mm, vias 8 -> 0
- net /H-Bridge-setup1/W2_B: track 40.5 -> 131.6 mm
- net Net-(U41-4A): track 90.8 -> 0.00 mm, vias 1 -> 0
- net Net-(U41-3A): track 86.0 -> 0.00 mm, vias 1 -> 0
- net Net-(U41-2A): track 71.6 -> 0.00 mm, vias 1 -> 0
- net Net-(U31-4A): track 66.7 -> 0.00 mm, vias 3 -> 0
- net /H-Bridge-setup1/W2_R: track 52.1 -> 115.9 mm, vias 1 -> 0
- net /H-Bridge-setup3/W2_B: track 13.9 -> 74.4 mm, vias 1 -> 0
- net Net-(U31-3A): track 59.4 -> 0.00 mm, vias 1 -> 0
- net Net-(U21-3A): track 58.3 -> 0.00 mm, vias 1 -> 0
- net /H-Bridge-setup4/W2_R: track 13.6 -> 71.1 mm
- net Net-(U41-1A): track 57.3 -> 0.00 mm, vias 3 -> 0
- net Net-(U11-3A): track 57.1 -> 0.00 mm, vias 3 -> 0
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Other:
- board size 99.6 x 64.3 mm -> 94.2 x 88.1 mm

Commit message: final design
Parts:
- removed H1: MountingHole, MountingHole:MountingHole_4.3mm_M4
- added G***: LOGO, Otter:LOGO, F.Cu at (164.1, 101.3)
- moved H4 0.25 mm to (235.7, 102.9)
- renumbered C12 to C1
Routing:
- net +5V: track 64.6 -> 413.3 mm, vias 0 -> 1
- net +12V: track 20.0 -> 324.8 mm, vias 0 -> 1
- net /H-Bridge-setup4/4A: track 0.00 -> 183.5 mm
- net /H-Bridge-setup4/3A: track 0.00 -> 150.1 mm, vias 0 -> 1
- net /H-Bridge-setup4/2A: track 0.00 -> 144.7 mm, vias 0 -> 1
- net /H-Bridge-setup4/1A: track 0.00 -> 123.4 mm, vias 0 -> 1
- net /H-Bridge-setup1/W2_B: track 131.6 -> 253.2 mm
- net /H-Bridge-setup3/2A: track 0.00 -> 116.4 mm
- net /H-Bridge-setup3/3A: track 0.00 -> 115.6 mm, vias 0 -> 1
- net /H-Bridge-setup3/4A: track 0.00 -> 112.4 mm
- net /H-Bridge-setup1/4A: track 0.00 -> 107.1 mm
- net /H-Bridge-setup1/3A: track 0.00 -> 101.6 mm, vias 0 -> 1
- net /H-Bridge-setup1/W2_R: track 115.9 -> 213.1 mm
- net /H-Bridge-setup2/3A: track 0.00 -> 84.9 mm, vias 0 -> 2
- net /H-Bridge-setup2/W1_R: track 78.9 -> 153.5 mm
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Other:
- outline, holes or cut-outs redrawn
- board text added: "5V GND 12V GND"
- board text added: "W1"
- board text added: "W2"
- board text added: "W3"
- board text added: "W4"
- board text added: "W5"
- board text added: "W6"
- board text added: "W7"
- board text added: "W8"
- board text added: "designed by PCBUILD3R"

Commit message: add version number
Other:
- board text added: "V1.0"
Changed lines of the file:
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@@
 		(capping no)
 		(filling no)
-		(zone_defaults)
 		(pcbplotparams
 			(layerselection 0x00000000_00000000_55555555_5755f5ff)
@@
 		)
 	)
+	(gr_text "V1.0"
+		(at 232.918 106.68 0)
+		(layer "B.SilkS")
+		(effects
+			(font
+				(size 1 1)
+				(thickness 0.1)
+			)
+			(justify left bottom mirror)
+		)
+	)
